File: hardware/VarioController/vc_board_v011.sch (EAGLE design)
At the start: 49 parts, among them IC1 WeMos D1 mini, IC2 MP2016DJ, IC3 DS3502U+, X1 SPTAF_1/3_3,5, X2 SPTAF_1/3_3,5, X3 SPTAF_1/3_3,5, X4 SPTAF_1/8_3,5, X5 05-JST-B5B-XH-A, X6 03-JST-B3B-XH-A

Commit message: Update PCB
Parts:
- removed C3, C4: 100n/25V, rcl:C-EUC0805
- removed C6: 4u7/50V, rcl:CPOL-EUD/7343-31W
- removed R16, R17, R18: (no value), rcl:R-EU_R0805
- added C15: 100n/25V, rcl:C-EUC0805
- added C19: 1000p/2KV, rcl:C-EUC1206K
- added D1: (no value), diode:DIODE-SMB
- added J1: (no value), con-lstb:MA03-1
- added R22, R23, R25: (no value), rcl:R-EU_R0805
- C1: value 100n/25V -> 1u/50V; device rcl:C-EUC0805 -> rcl:C-EUC1210K
- C7: value 1000p/2KV -> 4u7/50V; device rcl:C-EUC1206K -> rcl:CPOL-EUD/7343-31W
- C8: value 1000p/2KV -> 100n/25V; device rcl:C-EUC1206K -> rcl:C-EUC0805
- C9: value 1u/50V -> 100n/25V; device rcl:C-EUC1210K -> rcl:C-EUC0805
- R1: value (none) -> 120R
- R13, R14: value (none) -> 10K
- R2: value 120R -> (none)
- R3, R7: value 10K -> (none)
- renumbered R15 to R21, R19 to R24
Connections:
- removed net V-: C8.1, C9.1, LED1.C, PWS1.-VIN, R18.2, X4-2.KL
- new net N$7: C15.2, D1.C, IC1.5V
- new net N$8: J1.2, PWS1.REMOTE
- net +3V3: now also C9.2, R13.1, R14.1; no longer C3.2, R10.1, R9.1
- net +5V: now also C13.2, C19.2, D1.A, R1.1, R12.1, R22.1; no longer C1.2, C4.2, C7.2, IC1.5V, R14.1, R16.1, R2.1
- net AOUT: now also C10.2, C7.+; no longer C5.2, C6.+
- net ASET: now also C10.1; no longer C5.1
- net GND: now also C15.1, C5.1, C7.-, C8.1, C9.1, J1.1, LED1.C, PWS1.-VIN, R10.2, R4.2, R6.2, R9.1, X4-2.KL; no longer C10.1, C3.1, C4.1, C6.-, C8.2, R1.2, R3.1, R7.2
- net N$1: now also C5.2, R2.2, R3.2, R5.1; no longer C10.2, R1.1, R5.2, R6.2
- net N$10: now also R23.1; no longer R12.1
- net N$14: now also R22.2; no longer R14.2
- net N$15: now also R12.2; no longer R16.2
- net N$19: now also R25.1; no longer R13.1
- net N$2: now also R9.2; no longer R8.2
- net N$21: now also R5.2; no longer R4.2
- net N$3: now also R8.2; no longer R3.2
- net N$5: now also R1.2; no longer R2.2
- net N$6: now also R3.1; no longer R5.1
- net SCL: now also R14.2; no longer R10.2
- net SDA: now also R13.2; no longer R9.2
- net SHDN_REG: now also R10.1, R23.2; no longer R12.2, R7.1
- net UIN: now also R6.1, R7.2; no longer R17.2, R18.1
- net ULED2: now also R25.2; no longer R13.2
- net V+: now also C1.2, C19.1, C8.2, R2.1, R7.1; no longer C13.2, C7.1, C9.2, R17.1, R6.1
Other:
- moved on the sheet: C1, C10, C13, C5, C8, C9, R1, R10, R12, R13, R14, R2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

Commit message: PCB ORDER!
Parts:
- renumbered J1 to SJ1
Changed lines of the file:
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@@
 <?xml version="1.0" encoding="utf-8"?>
 <!DOCTYPE eagle SYSTEM "eagle.dtd">
-<eagle version="9.5.2">
+<eagle version="9.6.2">
 <drawing>
 <settings>
@@
 <part name="P+10" library="supply1" library_urn="urn:adsk.eagle:library:371" deviceset="V+" device=""/>
 <part name="D1" library="diode" library_urn="urn:adsk.eagle:library:210" deviceset="DIODE-" device="SMB" package3d_urn="urn:adsk.eagle:package:43404/2"/>
-<part name="J1" library="con-lstb" library_urn="urn:adsk.eagle:library:162" deviceset="MA03-1" device="" package3d_urn="urn:adsk.eagle:package:8339/1"/>
+<part name="SJ1" library="con-lstb" library_urn="urn:adsk.eagle:library:162" deviceset="MA03-1" device="" package3d_urn="urn:adsk.eagle:package:8339/1"/>
 <part name="GND22" library="supply1" library_urn="urn:adsk.eagle:library:371" deviceset="GND" device=""/>
 </parts>
@@
 <attribute name="VALUE" x="20.32" y="137.3886" size="1.778" layer="96"/>
 </instance>
-<instance part="J1" gate="G$1" x="48.26" y="66.04" smashed="yes">
+<instance part="SJ1" gate="G$1" x="48.26" y="66.04" smashed="yes">
 <attribute name="VALUE" x="46.99" y="58.42" size="1.778" layer="96"/>
 <attribute name="NAME" x="46.99" y="71.882" size="1.778" layer="95"/>
@@
 </segment>
 <segment>
-<pinref part="J1" gate="G$1" pin="1"/>
+<pinref part="SJ1" gate="G$1" pin="1"/>
 <pinref part="GND22" gate="1" pin="GND"/>
 <wire x1="55.88" y1="63.5" x2="60.96" y2="63.5" width="0.1524" layer="91"/>
@@
 <wire x1="71.12" y1="25.4" x2="63.5" y2="25.4" width="0.1524" layer="91"/>
 <wire x1="63.5" y1="25.4" x2="63.5" y2="66.04" width="0.1524" layer="91"/>
-<pinref part="J1" gate="G$1" pin="2"/>
+<pinref part="SJ1" gate="G$1" pin="2"/>
 <wire x1="55.88" y1="66.04" x2="63.5" y2="66.04" width="0.1524" layer="91"/>
 </segment>

Commit message: Update values
Parts:
- added FRAME1: MF_FRAMEDEFAULT, rca-frames:MF_FRAMEDEFAULT
- LED1, LED2: value (none) -> GN 2,65V/2mA; FARNELL_SKU (none) -> 2846598
- LED3: value (none) -> GE 1,85V/2mA; FARNELL_SKU (none) -> 2846596
- LED4: value (none) -> BL 2,65V/2mA; FARNELL_SKU (none) -> 2846594
- LED5: value (none) -> RT 1.95V/2mA; FARNELL_SKU (none) -> 2099241
- R12, R21: value (none) -> 10K
- R2: value (none) -> N/A
- R22: value (none) -> 1K2
- R23: value (none) -> 720R
- R24: value (none) -> 320R
- R25: value (none) -> 680R
- R3: value (none) -> 6K8
- R4: value (none) -> 3K2
- R5: value (none) -> 120R
Other:
- note added: "Widerstandswerte dimensioniert für 0 - 10 V Eingang."
- moved on the sheet: C11, C12, C13, C15, C19, C2, C5, C8, C9, D1, LED2, LED5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

Commit message: upd
Parts:
- R23: value 720R -> 680R
- R24: value 320R -> 330R
- R3: value 6K8 -> 6K8 0,1%
- R4: value 3K2 -> 3K1 0,1%
Changed lines of the file:
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@@
 <part name="P+5" library="supply1" library_urn="urn:adsk.eagle:library:371" deviceset="V+" device=""/>
 <part name="P+8" library="supply1" library_urn="urn:adsk.eagle:library:371" deviceset="V+" device=""/>
-<part name="R4" library="rcl" library_urn="urn:adsk.eagle:library:334" deviceset="R-EU_" device="R0805" package3d_urn="urn:adsk.eagle:package:23553/2" value="3K2"/>
+<part name="R4" library="rcl" library_urn="urn:adsk.eagle:library:334" deviceset="R-EU_" device="R0805" package3d_urn="urn:adsk.eagle:package:23553/2" value="3K1 0,1%"/>
 <part name="R5" library="rcl" library_urn="urn:adsk.eagle:library:334" deviceset="R-EU_" device="R0805" package3d_urn="urn:adsk.eagle:package:23553/2" value="120R"/>
-<part name="R3" library="rcl" library_urn="urn:adsk.eagle:library:334" deviceset="R-EU_" device="R0805" package3d_urn="urn:adsk.eagle:package:23553/2" value="6K8"/>
+<part name="R3" library="rcl" library_urn="urn:adsk.eagle:library:334" deviceset="R-EU_" device="R0805" package3d_urn="urn:adsk.eagle:package:23553/2" value="6K8 0,1%"/>
 <part name="R2" library="rcl" library_urn="urn:adsk.eagle:library:334" deviceset="R-EU_" device="R0805" package3d_urn="urn:adsk.eagle:package:23553/2" value="N/A"/>
 <part name="P+9" library="supply1" library_urn="urn:adsk.eagle:library:371" deviceset="V+" device=""/>
@@
 <attribute name="FARNELL_SKU" value="2099241"/>
 </part>
-<part name="R23" library="rcl" library_urn="urn:adsk.eagle:library:334" deviceset="R-EU_" device="R0805" package3d_urn="urn:adsk.eagle:package:23553/2" value="720R"/>
+<part name="R23" library="rcl" library_urn="urn:adsk.eagle:library:334" deviceset="R-EU_" device="R0805" package3d_urn="urn:adsk.eagle:package:23553/2" value="680R"/>
 <part name="R25" library="rcl" library_urn="urn:adsk.eagle:library:334" deviceset="R-EU_" device="R0805" package3d_urn="urn:adsk.eagle:package:23553/2" value="680R"/>
 <part name="GND18" library="supply1" library_urn="urn:adsk.eagle:library:371" deviceset="GND" device=""/>
@@
 <part name="X8" library="con-lstb" library_urn="urn:adsk.eagle:library:162" deviceset="MA03-1" device="" package3d_urn="urn:adsk.eagle:package:8339/1"/>
 <part name="GND20" library="supply1" library_urn="urn:adsk.eagle:library:371" deviceset="GND" device=""/>
-<part name="R24" library="rcl" library_urn="urn:adsk.eagle:library:334" deviceset="R-EU_" device="R0805" package3d_urn="urn:adsk.eagle:package:23553/2" value="320R"/>
+<part name="R24" library="rcl" library_urn="urn:adsk.eagle:library:334" deviceset="R-EU_" device="R0805" package3d_urn="urn:adsk.eagle:package:23553/2" value="330R"/>
 <part name="LED4" library="led" library_urn="urn:adsk.eagle:library:259" deviceset="LED" device="CHIPLED_0805" package3d_urn="urn:adsk.eagle:package:15821/2" value="BL 2,65V/2mA">
 <attribute name="FARNELL_SKU" value="2846594"/>
