File: hardware/VarioController/vc_board_v011.brd (EAGLE design)
At the start: 48.3 x 53.3 mm, 32 parts, among them IC1 WeMos D1 mini, K1 AQY21SOP, K2 AQY21SOP, K3 AQY21SOP, K4 AQY21SOP, X2 SPTAF_1/8_3,5, X3 05-JST-B5B-XH-A, X4 SPTAF_1/8_3,5

Commit message: Add layout
Parts:
- removed FRAME1: MF_FRAMEDEFAULT, rca-frames:MF_FRAME_DEFAULT
- removed K1, K2, K3, K4: AQY21SOP, relay:SOP04
- added C11, C12: (no value), rcl:D/7343-31W
- added C13: 100n/25V, rcl:C0805
- added IC2: MP2016DJ, mps-regulator:TSOT23-5
- added IC3: DS3502U+, maxim-ds3502:21-0061L_MXM
- added LED1, LED2, LED3, LED4, LED5: (no value), led:CHIPLED_0805
- added R13, R14, R15, R16, R17, R18, R19: (no value), rcl:R0805
- added R7: 10K, rcl:R0805
- added X5: 05-JST-B5B-XH-A, con-jst-xh:B5B-XH
- added X6: 03-JST-B3B-XH-A, con-jst-xh:B3B-XH
- added X7, X8: (no value), con-lstb:MA03-1
- C5: value (none) -> 100n/25V; device rcl:CT7343 -> rcl:C0805
- C6: value (none) -> 4u7/50V; device rcl:CT7343 -> rcl:D/7343-31W
- R1, R12, R4, R5, R6: value 220R -> (none)
- R10, R3, R8, R9: value 220R -> 10K
- R11: value 220R -> 1K3
- R2: value 220R -> 120R
- X1: value (none) -> SPTAF_1/3_3,5; device con-lstb:MA03-1 -> con-phoenix-sptaf:SPTAF_1/3_3,5
- X2: value SPTAF_1/8_3,5 -> SPTAF_1/3_3,5; device con-phoenix-sptaf:SPTAF_1/8_3,5 -> con-phoenix-sptaf:SPTAF_1/3_3,5
- X3: value 05-JST-B5B-XH-A -> SPTAF_1/3_3,5; device con-jst-xh:B5B-XH -> con-phoenix-sptaf:SPTAF_1/3_3,5
- moved C10 205.9 mm to (-40.0, -17.8), turned to 90 degrees
- moved R6 205.0 mm to (-44.5, -12.7)
- moved C8 199.1 mm to (-10.2, 12.1), turned to 180 degrees
- moved R2 196.3 mm to (-17.8, -33.0)
- moved R5 194.9 mm to (-44.5, -16.5)
- moved R4 187.8 mm to (-35.6, -16.5)
- moved R1 178.6 mm to (-44.5, -20.3), turned to 180 degrees
- moved C7 171.2 mm to (-10.2, -12.1), turned to 180 degrees
- moved PWS1 169.6 mm to (-10.2, 0.00), turned to 180 degrees
- moved C9 158.5 mm to (-10.8, -33.0), turned to 180 degrees
- moved R12 140.7 mm to (-31.8, 34.3), turned to 180 degrees
- moved C6 130.1 mm to (38.1, -36.8), turned to 90 degrees
- moved C5 126.4 mm to (33.7, -31.8), turned to 270 degrees
- moved X2 119.6 mm to (-38.1, 3.50), turned to 270 degrees
- moved R10 117.0 mm to (45.7, 1.91), turned to 180 degrees
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Connections:
- removed net N$11: K4.1, R12.1
- removed net N$12: R5.1, R6.2
- removed net N$20: IC1.12, R9.2
- removed net N$4: C8.1, C9.1, PWS1.2, PWS1.3, X4.2, X4.2A
- removed net N$7: K4.4, X2.4, X2.4A, X3.P$4
- removed net N$8: K3.4, X2.3, X2.3A, X3.P$3
- removed net N$9: K2.4, X2.2, X2.2A, X3.P$2
- new net AOUT: C5.2, C6.+, IC2.3, IC3.6, X4.3, X4.3A, X5.P$2
- new net ASET: C5.1, IC2.4, IC3.7, IC3.8, R11.1
- new net N$15: IC1.14, R16.2, X1.2, X1.2A, X2.2, X2.2A
- new net SCL: IC1.6, IC3.10, R10.2
- new net SDA: IC1.5, IC3.1, R9.2
- new net SHDN_REG: IC1.11, IC2.5, R12.2, R7.1
- new net UIN: IC1.13, R17.2, R18.1
- new net ULED1: IC1.4, LED4.C
- new net ULED2: IC1.3, R13.2
- new net V-: C8.1, C9.1, LED1.C, PWS1.2, PWS1.3, R18.2, X4.2, X4.2A
- net +3V3: now also IC3.3, R10.1, R19.2, R9.1, X7.2; no longer X1.2
- net +5V: now also C11.+, C12.+, R14.1, R16.1, X1.1, X1.1A, X2.1, X2.1A, X7.3; no longer C5.+, C6.+, R12.2, X1.3
- net GND: now also C11.-, C12.-, C13.1, IC2.2, IC3.2, IC3.4, IC3.5, LED2.C, LED3.C, LED5.C, R11.2, R7.2, X1.3, X1.3A, X2.3, X2.3A, X3.1, X3.1A, X4.4, X4.4A, X5.P$5, X7.1, X8.1; no longer C5.-, K1.2, K2.2, K3.2, X1.1, X2.8, X2.8A
- net N$1: now also R6.2; no longer X2.7, X2.7A
- net N$10: now also LED3.A, R12.1; no longer K1.4, X2.1, X2.1A, X3.P$1
- net N$13: now also LED1.A, R15.2; no longer K3.1, R11.1
- net N$14: now also LED2.A, R14.2; no longer K2.1, R10.1
- net N$16: now also IC1.8, X8.3; no longer K1.1, R9.1
- net N$17: now also IC1.7, X8.2; no longer IC1.15, K4.2
- net N$18: now also LED4.A, R19.1; no longer IC1.14, R11.2
- net N$19: now also LED5.A, R13.1; no longer IC1.13, R10.2
- net N$2: now also IC1.12, X4.6, X4.6A, X6.P$3; no longer IC1.4, X4.4, X4.4A
- net N$3: now also IC1.15, X4.5, X4.5A, X6.P$2; no longer IC1.3, X4.3, X4.3A
- net N$5: now also X4.7, X4.7A, X4.8, X4.8A, X6.P$1; no longer X4.5, X4.5A
- net N$6: now also R5.1, X3.2, X3.2A; no longer K1.3, K2.3, K3.3, K4.3, X2.5, X2.5A, X3.P$5
- net V+: now also C13.2, IC2.1, IC3.9, R15.1, R17.1, X3.3, X3.3A; no longer X2.6, X2.6A
Routing:
- net V+: track 0.00 -> 298.6 mm
- net +5V: track 131.5 -> 287.0 mm
- net SHDN_REG: track 0.00 -> 150.4 mm
- net V-: track 0.00 -> 144.8 mm, vias 0 -> 2
- net N$15: track 0.00 -> 133.0 mm
- net N$2: track 0.00 -> 127.2 mm
- net N$3: track 0.00 -> 120.4 mm
- net +3V3: track 56.3 -> 174.0 mm, vias 2 -> 3
- net N$21: track 0.00 -> 115.1 mm, vias 0 -> 1
- net AOUT: track 0.00 -> 100.7 mm
- net ULED2: track 0.00 -> 70.9 mm
- net ULED1: track 0.00 -> 66.9 mm
- net UIN: track 0.00 -> 57.5 mm, vias 0 -> 1
- net N$5: track 0.00 -> 56.9 mm
- net SCL: track 0.00 -> 45.0 mm
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Other:
- board size 48.3 x 53.3 mm -> 109.1 x 109 mm
- board text added: "#OpenPoolControl"
- board text added: "1-Wire"
- board text added: "100prznt.de"
- board text added: "2021"
- board text added: "5 V"
- board text added: "Date of manufacture"
- board text added: "ENABLE PUMP"
- board text added: "ERROR"
- board text added: "HW: 01.0"
- board text added: "PCB is optimized for fitting into a TK PC 1309-6-tm from the manufacturer SPELSBERG"
- board text added: "POWER"
- board text added: "Power"
- board text added: "Powerinput 12 - 36 VDC"
- board text added: "Pressure Sensor"
- board text added: "Pump"
- board text added: "Ruemmler, Elias"
- board text added: "STATUS"
- board text added: "Switch"
- board text added: "VarioControl"
- board text removed: "2020 HW: 01.0"
- board text removed: "Ruemmler, Elias 100prznt.de"
- board text removed: "Wifi2Dmx Bridge"

Commit message: Update PCB
Parts:
- removed C3, C4: 100n/25V, rcl:C0805
- removed C6: 4u7/50V, rcl:D/7343-31W
- removed R16, R17, R18: (no value), rcl:R0805
- added C15: 100n/25V, rcl:C0805
- added C19: 1000p/2KV, rcl:C1206K
- added D1: (no value), diode:SMB
- added J1: (no value), con-lstb:MA03-1
- added R22, R23, R25: (no value), rcl:R0805
- C1: value 100n/25V -> 1u/50V; device rcl:C0805 -> rcl:C1210K
- C7: value 1000p/2KV -> 4u7/50V; device rcl:C1206K -> rcl:D/7343-31W
- C8: value 1000p/2KV -> 100n/25V; device rcl:C1206K -> rcl:C0805
- C9: value 1u/50V -> 100n/25V; device rcl:C1210K -> rcl:C0805
- R1: value (none) -> 120R
- R13, R14: value (none) -> 10K
- R2: value 120R -> (none)
- R3, R7: value 10K -> (none)
- moved R14 85.7 mm to (43.8, 0.32), turned to 90 degrees
- moved C10 75.0 mm to (33.7, -31.8), turned to 270 degrees
- moved C5 75.0 mm to (-40.0, -17.8), turned to 90 degrees
- moved R13 74.8 mm to (40.0, 0.32), turned to 90 degrees
- moved C13 68.8 mm to (-32.4, 0.00)
- moved R12 65.4 mm to (33.0, 43.2), turned to 270 degrees
- moved C1 60.3 mm to (-10.8, -33.0)
- moved C8 57.6 mm to (27.3, -31.8), turned to 270 degrees
- moved C7 55.5 mm to (41.3, -33.0)
- moved R3 54.1 mm to (-44.5, -16.5), turned to 0 degrees
- moved R6 54.0 mm to (9.53, -13.3), turned to 270 degrees
- moved C9 51.4 mm to (39.4, -21.9), turned to 0 degrees
- moved C11 42.6 mm to (5.08, 14.0)
- moved R9 35.5 mm to (12.1, -21.6), turned to 270 degrees
- moved R10 34.0 mm to (27.3, -26.7), turned to 90 degrees
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- renumbered R15 to R21, R19 to R24
Connections:
- removed net V-: C8.1, C9.1, LED1.C, PWS1.2, PWS1.3, R18.2, X4.2, X4.2A
- new net N$7: C15.2, D1.C, IC1.1
- new net N$8: J1.2, PWS1.1
- net +3V3: now also C9.2, R13.1, R14.1; no longer C3.2, R10.1, R9.1
- net +5V: now also C13.2, C19.2, D1.A, R1.1, R12.1, R22.1; no longer C1.2, C4.2, C7.2, IC1.1, R14.1, R16.1, R2.1
- net AOUT: now also C10.2, C7.+; no longer C5.2, C6.+
- net ASET: now also C10.1; no longer C5.1
- net GND: now also C15.1, C5.1, C7.-, C8.1, C9.1, J1.1, LED1.C, PWS1.2, PWS1.3, R10.2, R4.2, R6.2, R9.1, X4.2, X4.2A; no longer C10.1, C3.1, C4.1, C6.-, C8.2, R1.2, R3.1, R7.2
- net N$1: now also C5.2, R2.2, R3.2, R5.1; no longer C10.2, R1.1, R5.2, R6.2
- net N$10: now also R23.1; no longer R12.1
- net N$14: now also R22.2; no longer R14.2
- net N$15: now also R12.2; no longer R16.2
- net N$19: now also R25.1; no longer R13.1
- net N$2: now also R9.2; no longer R8.2
- net N$21: now also R5.2; no longer R4.2
- net N$3: now also R8.2; no longer R3.2
- net N$5: now also R1.2; no longer R2.2
- net N$6: now also R3.1; no longer R5.1
- net SCL: now also R14.2; no longer R10.2
- net SDA: now also R13.2; no longer R9.2
- net SHDN_REG: now also R10.1, R23.2; no longer R12.2, R7.1
- net UIN: now also R6.1, R7.2; no longer R17.2, R18.1
- net ULED2: now also R25.2; no longer R13.2
- net V+: now also C1.2, C19.1, C8.2, R2.1, R7.1; no longer C13.2, C7.1, C9.2, R17.1, R6.1
Routing:
- net V-: track 144.8 -> 0.00 mm, vias 2 -> 0
- net AOUT: track 100.7 -> 83.4 mm
- net GND: track 20.0 -> 32.5 mm, vias 22 -> 13
- net V+: track 298.6 -> 287.2 mm
- net +5V: track 287.0 -> 276.7 mm
- net N$8: track 0.00 -> 9.42 mm
- net N$7: track 0.00 -> 8.27 mm
- net UIN: track 57.5 -> 64.0 mm
- net N$3: track 120.4 -> 115.8 mm
- net ULED2: track 70.9 -> 74.7 mm
- net SDA: track 40.6 -> 44.1 mm
- net N$15: track 133.0 -> 129.7 mm
- net SCL: track 45.0 -> 48.1 mm
- net +3V3: track 174.0 -> 171.2 mm
- net N$2: track 127.2 -> 124.6 mm
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Other:
- board size 109.1 x 109 mm -> 109 x 109 mm
- board text added: "0 - 10 V circuit"
- board text added: "1 2 3 1 2 3 1 2 3 1 2 3 4 5 6 7 8"
- board text added: "1-Wire (1)"
- board text added: "1-Wire (2)"
- board text added: "5 V (OK)"
- board text added: "5 V Data GND 5 V Data GND GND Signal (in) V+ V+ GND Signal (out) GND Mode 1 (in) Mode 2 (in) 5 V 5 V each pin 1 is marked"
- board text added: "HW: 01.1"
- board text added: "MADE IN GERMANY"
- board text added: "Mode Switch"
- board text added: "POWER (OK)"
- board text added: "Power Input"
- board text added: "Power Input 12 - 36 VDC"
- board text added: "Pump Ctrl"
- board text added: "SHDN DC/DC"
- board text added: "X1 X2 X3 X4"
- board text removed: "1-Wire"
- board text removed: "5 V"
- board text removed: "HW: 01.0"
- board text removed: "POWER"
- board text removed: "Power"
- board text removed: "Powerinput 12 - 36 VDC"
- board text removed: "Pump"
- board text removed: "Switch"

Commit message: update layout
Parts:
- moved LED1 5.08 mm to (-21.6, 47.0)
- moved LED2 5.08 mm to (-21.6, 40.6)
- moved LED3 5.08 mm to (-21.6, 34.3)
- moved LED4 5.08 mm to (-21.6, 27.9)
- moved LED5 5.08 mm to (-21.6, 21.6)
- moved C7 0.63 mm to (40.6, -33.0)
Routing:
- net GND: track 32.5 -> 18.1 mm, vias 13 -> 12
- net ULED1: track 68.9 -> 63.8 mm
- net N$19: track 3.08 -> 8.16 mm
- net N$18: track 3.08 -> 8.16 mm
- net N$14: track 3.08 -> 8.16 mm
- net N$13: track 3.08 -> 8.16 mm
- net N$10: track 3.08 -> 8.16 mm
- net N$21: track 115.1 -> 114.3 mm
- net AOUT: track 83.4 -> 84.0 mm

Commit message: PCB ORDER!
Parts:
- moved R21 30.5 mm to (-40.6, 17.8), turned to 90 degrees
- moved R22 23.7 mm to (-38.1, 17.8), turned to 90 degrees
- moved R23 16.9 mm to (-35.6, 17.8), turned to 270 degrees
- moved R24 10.2 mm to (-32.4, 17.8), turned to 270 degrees
- moved R1 5.24 mm to (-16.5, -27.9), turned to 270 degrees
- moved R25 4.26 mm to (-29.8, 17.8), turned to 270 degrees
- renumbered J1 to SJ1
Routing:
- net V+: track 287.2 -> 246.7 mm
- net N$13: track 8.16 -> 35.8 mm
- net N$14: track 8.16 -> 28.3 mm
- net N$10: track 8.16 -> 20.9 mm
- net +3V3: track 171.2 -> 162.9 mm, vias 3 -> 5
- net N$18: track 8.16 -> 14.9 mm
- net SHDN_REG: track 150.6 -> 156.7 mm
- net N$15: track 129.7 -> 134.5 mm
- net N$5: track 56.9 -> 60.9 mm
- net N$21: track 114.3 -> 112.1 mm
- net N$6: track 27.2 -> 25.2 mm
- net ULED2: track 74.7 -> 76.7 mm
- net ULED1: track 63.8 -> 65.3 mm
- net +5V: track 276.7 -> 275.5 mm
- net N$19: track 8.16 -> 8.95 mm
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Other:
- board text added: "96 x 96 mm 109 x 109 mm"
- board text added: "Distance mounting holes PCB dimensions"
- board text added: "JLC order ID"
- board text added: "JLCJLCJLCJLC"
- board text added: "POWER"
- board text added: "Terminal assignment"
- board text removed: "POWER (OK)"

Commit message: Update values
Parts:
- added FRAME1: MF_FRAMEDEFAULT, rca-frames:MF_FRAME_DEFAULT
- LED1, LED2: value (none) -> GN 2,65V/2mA
- LED3: value (none) -> GE 1,85V/2mA
- LED4: value (none) -> BL 2,65V/2mA
- LED5: value (none) -> RT 1.95V/2mA
- R12, R21: value (none) -> 10K
- R2: value (none) -> N/A
- R22: value (none) -> 1K2
- R23: value (none) -> 720R
- R24: value (none) -> 320R
- R25: value (none) -> 680R
- R3: value (none) -> 6K8
- R4: value (none) -> 3K2
- R5: value (none) -> 120R
