File: hardware/VarioController/vc_board_v011.brd (EAGLE design)
At the start: 109 x 109 mm, 51 parts, among them IC1 WeMos D1 mini, IC2 MP2016DJ, IC3 DS3502U+, X1 SPTAF_1/3_3,5, X2 SPTAF_1/3_3,5, X3 SPTAF_1/3_3,5, X4 SPTAF_1/8_3,5, X5 05-JST-B5B-XH-A, X6 03-JST-B3B-XH-A

Commit message: upd
Parts:
- R23: value 720R -> 680R
- R24: value 320R -> 330R
- R3: value 6K8 -> 6K8 0,1%
- R4: value 3K2 -> 3K1 0,1%
Changed lines of the file:
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@@
 <attribute name="VALUE" x="-9.195" y="-30.445" size="1.016" layer="27" rot="R180"/>
 </element>
-<element name="R4" library="rcl" library_urn="urn:adsk.eagle:library:334" package="R0805" package3d_urn="urn:adsk.eagle:package:23553/2" value="3K2" x="-44.45" y="-19.05" smashed="yes" rot="R180">
+<element name="R4" library="rcl" library_urn="urn:adsk.eagle:library:334" package="R0805" package3d_urn="urn:adsk.eagle:package:23553/2" value="3K1 0,1%" x="-44.45" y="-19.05" smashed="yes" rot="R180">
 <attribute name="NAME" x="-46.6725" y="-18.415" size="1.27" layer="25" rot="R180"/>
 <attribute name="POPULARITY" value="86" x="-44.45" y="-19.05" size="1.778" layer="27" rot="R180" display="off"/>
@@
 <attribute name="VALUE" x="-36.195" y="-19.05" size="1.27" layer="27"/>
 </element>
-<element name="R3" library="rcl" library_urn="urn:adsk.eagle:library:334" package="R0805" package3d_urn="urn:adsk.eagle:package:23553/2" value="6K8" x="-44.45" y="-16.51" smashed="yes">
+<element name="R3" library="rcl" library_urn="urn:adsk.eagle:library:334" package="R0805" package3d_urn="urn:adsk.eagle:package:23553/2" value="6K8 0,1%" x="-44.45" y="-16.51" smashed="yes">
 <attribute name="NAME" x="-46.6725" y="-15.875" size="1.27" layer="25" rot="R180"/>
 <attribute name="POPULARITY" value="86" x="-44.45" y="-16.51" size="1.778" layer="27" display="off"/>
@@
 <attribute name="VALUE" x="-22.86" y="19.05" size="1.27" layer="27"/>
 </element>
-<element name="R23" library="rcl" library_urn="urn:adsk.eagle:library:334" package="R0805" package3d_urn="urn:adsk.eagle:package:23553/2" value="720R" x="-35.56" y="17.78" smashed="yes" rot="R270">
+<element name="R23" library="rcl" library_urn="urn:adsk.eagle:library:334" package="R0805" package3d_urn="urn:adsk.eagle:package:23553/2" value="680R" x="-35.56" y="17.78" smashed="yes" rot="R270">
 <attribute name="NAME" x="-36.195" y="15.5575" size="1.27" layer="25" rot="R270"/>
 <attribute name="POPULARITY" value="86" x="-35.56" y="17.78" size="1.778" layer="27" rot="R270" display="off"/>
@@
 <attribute name="VALUE" x="48.641" y="5.715" size="1.27" layer="27" ratio="10" rot="R90"/>
 </element>
-<element name="R24" library="rcl" library_urn="urn:adsk.eagle:library:334" package="R0805" package3d_urn="urn:adsk.eagle:package:23553/2" value="320R" x="-32.385" y="17.78" smashed="yes" rot="R270">
+<element name="R24" library="rcl" library_urn="urn:adsk.eagle:library:334" package="R0805" package3d_urn="urn:adsk.eagle:package:23553/2" value="330R" x="-32.385" y="17.78" smashed="yes" rot="R270">
 <attribute name="NAME" x="-33.02" y="15.5575" size="1.27" layer="25" rot="R270"/>
 <attribute name="POPULARITY" value="86" x="-32.385" y="17.78" size="1.778" layer="27" rot="R270" display="off"/>
